File: Group Project PCB Updated.brd (EAGLE design)
At the start: 12 parts, among them J2 1X04_SMD_STRAIGHT_COMBO, J3 1x3 RA Female .1", J4 1X04_SMD_STRAIGHT_COMBO, J5 1X04_SMD_STRAIGHT_COMBO, J7 1X04_SMD_STRAIGHT_COMBO, J8 1x3 RA Female .1"

Commit message: Add files via upload
Parts:
- added J1: (no value), EENG3110 V1 Library:1X05_LONGPADS
- moved R2 151.2 mm to (12.7, -36.8), turned to 180 degrees
- moved T1 134.1 mm to (-3.81, -38.1)
- moved SG1 128.3 mm to (-2.54, -26.7)
- moved C2 124.8 mm to (1.27, -48.3)
- moved J8 124.0 mm to (50.8, -34.3), turned to 270 degrees
- moved R1 123.4 mm to (3.81, -58.4), turned to 180 degrees
- moved J3 108.9 mm to (47.0, -43.2), turned to 270 degrees
- moved J5 92.0 mm to (17.8, -29.2), turned to 180 degrees
- moved J7 90.9 mm to (33.0, -49.5), turned to 180 degrees
- moved J2 75.4 mm to (30.5, -40.6), turned to 180 degrees
- moved J4 71.2 mm to (30.5, -33.0), turned to 180 degrees
Connections:
- new net N$19: IC1.7, J1.4
- new net N$20: IC1.8, J1.3
- new net N$21: IC1.17, J1.2
- net +5V: now also J1.1
- net GND: now also J1.5
- net N$12: now also IC1.15, J8.1; no longer IC1.18, R2.1
- net N$13: now also IC1.16; no longer IC1.23
- net N$14: now also R2.1; no longer J8.1
- net N$16: now also J8.3; no longer J8.2
- net N$18: now also J8.2; no longer J8.3
- net N$3: now also IC1.23, J4.3; no longer IC1.21, J4.2
- net N$4: now also J4.2; no longer J4.3
- net N$5: now also IC1.21, J2.3; no longer IC1.19, J2.2
- net N$6: now also J2.2; no longer J2.3
- net N$7: now also IC1.19, J7.3; no longer IC1.8, J7.2
- net N$8: now also IC1.18, J7.2; no longer IC1.7, J7.3
Routing:
- net GND: track 0.00 -> 110.4 mm
- net +5V: track 0.00 -> 79.7 mm
- net N$7: track 0.00 -> 38.9 mm
- net N$21: track 0.00 -> 38.8 mm
- net N$8: track 0.00 -> 36.7 mm
- net N$18: track 0.00 -> 31.4 mm
- net N$5: track 0.00 -> 31.4 mm
- net N$6: track 0.00 -> 29.0 mm
- net N$13: track 0.00 -> 27.7 mm
- net N$16: track 0.00 -> 24.7 mm
- net N$14: track 0.00 -> 22.5 mm
- net N$2: track 0.00 -> 22.3 mm
- net N$15: track 0.00 -> 20.8 mm
- net N$12: track 0.00 -> 20.1 mm
- net N$11: track 0.00 -> 19.7 mm
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